File: Control PCB/Control PCB.kicad_pcb (KiCad board)
At the start: 2 copper layers, 65.5 x 60.8 mm, 27 parts, among them J1 L_Motor_XT30_F, J2 R_Motor_XT30_F, J3 Motor_Power_XT30_M, J4 Sense_L, J5 Sense_R, J6 Amp_power_XT30_M, Q1 IRLZ44N, Q2 IRLZ44N, U1 TL071, U2 TL071

Commit message: Add files via upload
Parts:
- added C10: 10u, Capacitor_THT:C_Rect_L4.6mm_W2.0mm_P2.50mm_MKS02_FKP02, F.Cu at (36.5, 41.2)
- added C11: 10u, Capacitor_THT:C_Rect_L4.6mm_W2.0mm_P2.50mm_MKS02_FKP02, F.Cu at (36.5, 50.2)
- added C7: 10u, Capacitor_THT:C_Rect_L4.6mm_W2.0mm_P2.50mm_MKS02_FKP02, F.Cu at (37.0, 32.5)
- added C8: 10u, Capacitor_THT:C_Rect_L4.6mm_W2.0mm_P2.50mm_MKS02_FKP02, F.Cu at (37.0, 56.5)
- added C9: 10u, Capacitor_THT:C_Rect_L4.6mm_W2.0mm_P2.50mm_MKS02_FKP02, F.Cu at (65.5, 43.5)
- added D3: 1N4001, Diode_THT:D_DO-41_SOD81_P10.16mm_Horizontal, F.Cu at (37.1, 35.5)
- added D4: 1N4001, Diode_THT:D_DO-41_SOD81_P10.16mm_Horizontal, F.Cu at (37.1, 53.5)
- Q1, Q2: footprint Package_TO_SOT_THT:TO-220-3_Vertical -> Package_TO_SOT_THT:TO-220-3_Horizontal_TabDown
- moved R2 41.3 mm to (45.4, 69.5), turned to 0 degrees
- moved R3 41.2 mm to (45.4, 19.8), turned to 0 degrees
- moved R7 16.2 mm to (27.0, 69.2), turned to 90 degrees
- moved C6 14.7 mm to (29.2, 56.5)
- moved U2 14.4 mm to (37.3, 67.3), turned to 180 degrees
- moved C5 14.0 mm to (20.8, 60.2), turned to -90 degrees
- moved C3 13.1 mm to (20.8, 28.5), turned to 90 degrees
- moved J4 12.7 mm to (22.0, 20.2)
- moved J5 12.3 mm to (22.0, 66.0)
- moved Q2 8.59 mm to (65.0, 54.6), turned to 180 degrees
- moved C4 8.38 mm to (26.8, 32.5)
- moved R6 7.52 mm to (23.8, 25.9), turned to -90 degrees
- moved Q1 5.24 mm to (59.9, 34.7)
- moved R4 5.24 mm to (62.0, 41.9)
- moved R1 5.06 mm to (58.8, 47.3)
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Connections:
- C4 pad 2: Sense_L -> Net-(D3-A)
- C6 pad 1: Sense_R -> Net-(D4-A)
- R6 pad 2: Sense_L -> Net-(D3-A)
- R8 pad 2: Sense_R -> Net-(D4-A)
- U1 pad 6: Sense_L -> Net-(D3-A)
- U2 pad 6: Sense_R -> Net-(D4-A)
Routing:
- net +BATT: track 77.2 -> 8.11 mm, vias 0 -> 4
- net +9V: track 41.5 -> 0.00 mm
- net -9V: track 37.9 -> 0.00 mm
- net PWM_R: track 9.74 -> 44.1 mm
- net Net-(D3-A): track 0.00 -> 17.7 mm
- net Net-(D4-A): track 0.00 -> 14.2 mm
- net Sense_R: track 32.9 -> 19.5 mm
- net Net-(J4-Pin_1): track 15.4 -> 5.18 mm
- net Net-(D1-A): track 19.1 -> 27.0 mm, vias 0 -> 90
- net Sense_L: track 13.0 -> 6.05 mm
- net Net-(U1--): track 14.6 -> 9.59 mm
- net PWM_L: track 20.4 -> 24.7 mm
- net Net-(D2-A): track 26.9 -> 30.3 mm, vias 0 -> 90
- net Net-(U2--): track 14.5 -> 17.4 mm
- net Net-(C3-Pad1): track 10.8 -> 9.47 mm
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- added copper zone on In1.Cu, net +9V
- added copper zone on F.Cu, net +BATT
- added copper zone on In2.Cu, net -9V
- added copper zone on B.Cu, net Net-(D1-A)
- added copper zone on F.Cu, net Net-(D1-A)
- added copper zone on In1.Cu, net Net-(D1-A)
- added copper zone on In2.Cu, net Net-(D1-A)
- added copper zone on B.Cu, net Net-(D2-A)
- added copper zone on F.Cu, net Net-(D2-A)
- added copper zone on In1.Cu, net Net-(D2-A)
- added copper zone on In2.Cu, net Net-(D2-A)
- removed copper zone on F.Cu, net GND
Other:
- copper layers 2 -> 4
